File: PCB/ergodash.kicad_pcb (KiCad board)
At the start: 2 copper layers, 149.9 x 127.4 mm, 86 parts, among them SW1 SW_PUSH, SW10 SW_PUSH, SW11 SW_PUSH, SW12 SW_PUSH, SW13 SW_PUSH, SW14 SW_PUSH, SW15 SW_PUSH, SW16 SW_PUSH, SW17 SW_PUSH, SW18 SW_PUSH, SW19 SW_PUSH, SW2 SW_PUSH, SW20 SW_PUSH, SW21 SW_PUSH, SW22 SW_PUSH, SW23 SW_PUSH, SW24 SW_PUSH, SW25 SW_PUSH, SW26 SW_PUSH, SW27 SW_PUSH, SW28 SW_PUSH, SW3 SW_PUSH, SW30 SW_PUSH, SW31 SW_PUSH, SW32 SW_PUSH, SW33 SW_PUSH, SW34 SW_PUSH, SW35 SW_PUSH, SW36 SW_PUSH, SW38 SW_PUSH, SW39 SW_PUSH, SW4 SW_PUSH, SW40 SW_PUSH, SW41 SW_PUSH, SW5 SW_PUSH, SW6 SW_PUSH, SW7 SW_PUSH, SW8 SW_PUSH, SW9 SW_PUSH

Commit message: temp
Parts:
- added C1: MountingHole, ergodash_2040:Plate_MountingHole_cut, F.Cu at (80.9, 140.3)
- added C2: MountingHole, ergodash_2040:Plate_MountingHole_cut, F.Cu at (209.5, 161.5)
- added C3: MountingHole, ergodash_2040:Plate_MountingHole_cut, F.Cu at (129.7, 140.3)
- added C4: MountingHole, ergodash_2040:Plate_MountingHole_cut, F.Cu at (176.5, 142.5)
- added C5: MountingHole, ergodash_2040:Plate_MountingHole_cut, F.Cu at (225.1, 134.5)
- added C6: MountingHole, ergodash_2040:Plate_MountingHole_cut, F.Cu at (164.6, 163.6)
- added C7: MountingHole, ergodash_2040:Plate_MountingHole_cut, F.Cu at (146.6, 162.1)
- added C8: MountingHole, ergodash_2040:Plate_MountingHole_cut, F.Cu at (138.6, 162.1)
- SW1, SW2, SW3, SW30, SW4: footprint ergodash_2040:Kailh_socket_MX -> ergodash_2040:Kailh_socket_MX_leftmost
- SW25, SW26, SW27, SW28: footprint ergodash_2040:Kailh_socket_MX -> ergodash_2040:Kailh_socket_MX_rightmost
- moved D33 4.72 mm to (171.8, 138.4), turned to 150 degrees
- moved D30 0.56 mm to (106.5, 138.4)
- moved D34 0.40 mm to (182.7, 140.3)
- turned LED10 to 180 degrees
- turned LED11 to 180 degrees
- turned LED12 to 180 degrees
Routing:
- net VCC: track 3.23 -> 371.2 mm, vias 1 -> 16
- net /col5: track 86.3 -> 57.1 mm
- net Net-(LED10-Pad4): track 0.00 -> 26.1 mm, vias 0 -> 1
- net Net-(LED11-Pad2): track 0.00 -> 23.8 mm, vias 0 -> 2
- net Net-(LED10-Pad2): track 0.00 -> 22.1 mm, vias 0 -> 1
- net Net-(LED8-Pad2): track 27.7 -> 6.85 mm, vias 0 -> 2
- net Net-(LED1-Pad2): track 17.9 -> 6.79 mm, vias 0 -> 2
- net Net-(LED3-Pad2): track 17.9 -> 28.2 mm, vias 0 -> 2
- net Net-(LED2-Pad2): track 17.9 -> 26.9 mm, vias 0 -> 2
- net Net-(LED5-Pad2): track 18.7 -> 27.7 mm, vias 0 -> 2
- net Net-(LED6-Pad2): track 18.7 -> 27.4 mm, vias 0 -> 2
- net /row4: track 90.4 -> 83.5 mm
- net GND: track 6.16 -> 13.0 mm, vias 2 -> 4
- net Net-(D28-Pad2): track 20.7 -> 17.0 mm, vias 1 -> 0
- net unconnected-(LED12-Pad2): track 0.00 -> 3.42 mm, vias 0 -> 1
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