File: PCB/ergodash.kicad_sch (KiCad schematic)
At the start: 86 parts, among them SW1 SW_PUSH, SW10 SW_PUSH, SW11 SW_PUSH, SW12 SW_PUSH, SW13 SW_PUSH, SW14 SW_PUSH, SW15 SW_PUSH, SW16 SW_PUSH, SW17 SW_PUSH, SW18 SW_PUSH, SW19 SW_PUSH, SW2 SW_PUSH, SW20 SW_PUSH, SW21 SW_PUSH, SW22 SW_PUSH, SW23 SW_PUSH, SW24 SW_PUSH, SW25 SW_PUSH, SW26 SW_PUSH, SW27 SW_PUSH, SW28 SW_PUSH, SW3 SW_PUSH, SW30 SW_PUSH, SW31 SW_PUSH, SW32 SW_PUSH, SW33 SW_PUSH, SW34 SW_PUSH, SW35 SW_PUSH, SW36 SW_PUSH, SW38 SW_PUSH, SW39 SW_PUSH, SW4 SW_PUSH, SW40 SW_PUSH, SW41 SW_PUSH, SW5 SW_PUSH, SW6 SW_PUSH, SW7 SW_PUSH, SW8 SW_PUSH, SW9 SW_PUSH

Commit message: temp
Parts:
- LED1, LED10, LED11, LED12, LED2, LED3, LED4, LED5, LED6, LED7, LED8, LED9: footprint ergodash_2040:LED_WS2812B_reversible -> ergodash_2040:WS2812B-5
Connections:
- net RBG: now also LED1.4 (DIN)
- net col4: now also SW34.2; no longer SW34.1
- net at D33.2 (A): now also SW34.1; no longer SW34.2
Other:
- moved on the sheet: SW34

Commit message: temp
Parts:
- added C1, C2, C3, C4, C5, C6, C7, C8, C9: MountingHole, ergodash_2040:Plate_MountingHole_cut, symbol Mechanical:MountingHole
- added J1: Conn_01x04, symbol Connector_Generic:Conn_01x04
- added J2: Conn_01x15, Connector_FFC-FPC:Molex_502244-1530_1x15-1MP_P0.5mm_Horizontal, symbol Connector_Generic:Conn_01x15
- SW1, SW2, SW3, SW30, SW4: footprint ergodash_2040:Kailh_socket_MX -> ergodash_2040:Kailh_socket_MX_leftmost
- SW25, SW26, SW27, SW28: footprint ergodash_2040:Kailh_socket_MX -> ergodash_2040:Kailh_socket_MX_rightmost
Connections:
- net GND: now also J2.1 (Pin_1), J2.15 (Pin_15)
- net RBG: now also J2.14 (Pin_14)
- net VCC: now also J1.3 (Pin_3), J1.4 (Pin_4)
- net col0: now also J2.2 (Pin_2)
- net col1: now also J2.3 (Pin_3)
- net col2: now also J2.4 (Pin_4)
- net col3: now also J2.5 (Pin_5)
- net col4: now also J2.6 (Pin_6)
- net col5: now also J2.7 (Pin_7)
- net col6: now also J2.8 (Pin_8)
- net row0: now also J2.13 (Pin_13)
- net row1: now also J2.12 (Pin_12)
- net row2: now also J2.11 (Pin_11)
- net row3: now also J2.10 (Pin_10)
- net row4: now also J2.9 (Pin_9)
