File: PCB/ioparts/usb_c/usb_type_c.kicad_pcb (KiCad board)
At the start: 2 copper layers, 20 x 14.5 mm, 9 parts, among them J2 USB_C_Receptacle_USB2.0, J4 Conn_01x04

Commit message: misc pcbs
Parts:
- added J1: Conn_01x04, Connector_JST:JST_SH_SM04B-SRSS-TB_1x04-1MP_P1.00mm_Horizontal, F.Cu at (100.0, 71.4)
- moved J4 2.50 mm to (97.0, 67.4)
- turned R1 to -90 degrees
- turned R2 to -90 degrees
Routing:
- net Net-(J2-PadB5): track 7.36 -> 9.08 mm
- net Net-(J2-PadA5): track 8.03 -> 9.45 mm
- net VBUS_C: track 13.3 -> 14.4 mm, vias 2 -> 1
- net DP_C: track 9.15 -> 8.56 mm
Other:
- board size 20 x 14.5 mm -> 20 x 15.5 mm
- board text removed: "D+"
- board text removed: "D-"
- board text removed: "GND"
- board text removed: "VBUS"
