File: PCB/rp2040_zero_controller/rp2040_zero.kicad_pcb (KiCad board)
At the start: 2 copper layers, 39 x 32.7 mm, 15 parts, among them J1 Conn_01x04, J2 Conn_01x04, J3 Conn_01x04, J4 Conn_01x12, J5 Conn_01x04, U1 rp2040_zero, U2 74AHCT1G125, U3 74AHCT1G125

Commit message: temp
Parts:
- removed H3, H4: MountingHole, MountingHole:MountingHole_2.1mm
- removed U3: 74AHCT1G125, Package_TO_SOT_SMD:SOT-23-5_HandSoldering
- J4: footprint ergodash_controller:HDGC_1.0K-J-12PW -> Connector_FFC-FPC:Molex_200528-0120_1x12-1MP_P1.00mm_Horizontal; moved to F.Cu
- moved U2 28.5 mm to (115.4, 124.7)
- moved R2 14.8 mm to (86.4, 125.8), turned to 0 degrees
- moved R3 13.5 mm to (82.7, 124.7), turned to -90 degrees
- moved J1 12.9 mm to (114.5, 130.8), turned to 0 degrees
- moved J2 12.8 mm to (115.0, 118.0), turned to 90 degrees
- moved R1 12.4 mm to (86.4, 123.5), turned to 0 degrees
- moved H1 6.26 mm to (86.5, 111.5)
- moved H2 6.26 mm to (113.5, 111.5)
- moved J4 1.36 mm to (100.0, 130.0)
- moved J5 1.28 mm to (85.0, 118.0)
- moved J3 1.00 mm to (85.5, 130.8)
Connections:
- J1 pad 3: SDA -> VCC
- J1 pad 4: SCL -> RGB_5v_2
- J2 pad 3: VCC -> SDA
- J2 pad 4: RGB_5v -> SCL
- R1 pad 2: SDA -> SCL
- R2 pad 2: SCL -> SDA
- R3 pad 1: Handness -> +3V3
- R3 pad 2: +3V3 -> Handness
- U1 pad 10: GP8 -> GP7
- U1 pad 11: GP5 -> GP6
- U1 pad 12: GP3 -> GP5
- U1 pad 13: GP1 -> GP4
- U1 pad 14: GP2 -> GP3
- U1 pad 15: GP4 -> GP2
- U1 pad 26: GP6 -> GP1
- U1 pad 27: RGB2 -> Handness
- U1 pad 28: Handness -> unconnected-(U1-Pad28)
- U1 pad 5: GP7 -> GP12
- U1 pad 6: GP9 -> GP11
- U1 pad 7: GP11 -> GP10
- U1 pad 8: GP12 -> GP9
- U1 pad 9: GP10 -> GP8
- U2 pad 2: RGB2 -> RGB
Routing:
- net RGB_5v_2: track 5.25 -> 34.8 mm, vias 0 -> 2
- net GND: track 16.2 -> 1.49 mm, vias 19 -> 13
- net GP6: track 17.8 -> 3.46 mm
- net +3V3: track 9.41 -> 23.6 mm
- net RGB2: track 11.1 -> 0.00 mm
- net GP7: track 15.7 -> 4.80 mm
- net RGB_5v: track 9.47 -> 0.00 mm
- net GP1: track 5.37 -> 14.8 mm
- net GP4: track 13.5 -> 5.03 mm
- net GP10: track 6.52 -> 13.7 mm
- net GP11: track 9.08 -> 16.1 mm
- net Handness: track 10.2 -> 16.1 mm
- net SDA: track 51.0 -> 56.5 mm, vias 1 -> 3
- net GP3: track 4.99 -> 9.74 mm
- net GP9: track 12.4 -> 8.49 mm
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Other:
- board size 39 x 32.7 mm -> 37 x 32.7 mm

Commit message: temp
Parts:
- J4: footprint Connector_FFC-FPC:Molex_200528-0120_1x12-1MP_P1.00mm_Horizontal -> ergodash_controller:CF50121D0R0-10-NH
Changed lines of the file:
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@@
     )
   )
-  (footprint "Connector_FFC-FPC:Molex_200528-0120_1x12-1MP_P1.00mm_Horizontal" (layer "F.Cu")
+  (footprint "ergodash_controller:CF50121D0R0-10-NH" (layer "F.Cu")
     (at 100 130)
-    (descr "Molex Molex 1.00mm Pitch Easy-On BackFlip, Right-Angle, Bottom Contact FFC/FPC, 200528-0120, 12 Circuits (https://www.molex.com/pdm_docs/sd/2005280120_sd.pdf), generated with kicad-footprint-generator")
-    (tags "connector Molex  top entry")
     (property "Sheetfile" "rp2040_zero.kicad_sch")
     (property "Sheetname" "")
     (attr smd)
-    (fp_text reference "J4" (at 0 -2.61) (layer "F.SilkS") hide
+    (fp_text reference "J4" (at 1 -0.5 unlocked) (layer "F.SilkS")
       (effects (font (size 1 1) (thickness 0.15)))
     )
-    (fp_text value "Conn_01x12" (at 0 5.39) (layer "F.Fab")
+    (fp_text value "Conn_01x12" (at 1 1 unlocked) (layer "F.Fab")
       (effects (font (size 1 1) (thickness 0.15)))
     )
-    (fp_text user "${REFERENCE}" (at 0 1.39) (layer "F.Fab") hide
+    (fp_text user "${REFERENCE}" (at 1 2.5 unlocked) (layer "F.Fab")
       (effects (font (size 1 1) (thickness 0.15)))
     )
-    (fp_line (start 7.91 3) (end 8.71 3) (layer "F.SilkS") (width 0.12))
-    (fp_line (start -8.71 2.7) (end -8.71 3) (layer "F.SilkS") (width 0.12))
-    (fp_line (start -5.96 -0.82) (end -7.94 -0.82) (layer "F.SilkS") (width 0.12))
-    (fp_line (start -7.94 -1.17) (end -8.71 -1.17) (layer "F.SilkS") (width 0.12))
-    (fp_line (start -8.71 3) (end -7.91 3) (layer "F.SilkS") (width 0.12))
-    (fp_line (start 8.71 -1.17) (end 7.94 -1.17) (layer "F.SilkS") (width 0.12))
-    (fp_line (start -7.94 -0.82) (end -7.94 -1.17) (layer "F.SilkS") (width 0.12))
-    (fp_line (start -8.71 -1.17) (end -8.71 0.88) (layer "F.SilkS") (width 0.12))
-    (fp_line (start 7.94 -0.82) (end 5.96 -0.82) (layer "F.SilkS") (width 0.12))
-    (fp_line (start 8.71 0.88) (end 8.71 -1.17) (layer "F.SilkS") (width 0.12))
-    (fp_line (start -7.91 4.3) (end 7.91 4.3) (layer "F.SilkS") (width 0.12))
-    (fp_line (start 7.94 -1.17) (end 7.94 -0.82) (layer "F.SilkS") (width 0.12))
-    (fp_line (start 7.91 4.3) (end 7.91 3) (layer "F.SilkS") (width 0.12))
-    (fp_line (start 8.71 3) (end 8.71 2.7) (layer "F.SilkS") (width 0.12))
-    (fp_line (start -7.91 3) (end -7.91 4.3) (layer "F.SilkS") (width 0.12))
-    (fp_line (start -5.96 -1.41) (end -5.96 -0.82) (layer "F.SilkS") (width 0.12))
-    (fp_line (start -9.8 -1.91) (end -9.8 4.69) (layer "F.CrtYd") (width 0.05))
-    (fp_line (start 9.8 -1.91) (end -9.8 -1.91) (layer "F.CrtYd") (width 0.05))
-    (fp_line (start 9.8 4.69) (end 9.8 -1.91) (layer "F.CrtYd") (width 0.05))
-    (fp_line (start -9.8 4.69) (end 9.8 4.69) (layer "F.CrtYd") (width 0.05))
-    (fp_line (start 8.05 -0.71) (end -8.05 -0.71) (layer "F.Fab") (width 0.1))
-    (fp_line (start 7.8 0.19) (end -7.8 0.19) (layer "F.Fab") (width 0.1))
-    (fp_line (start 7.8 4.19) (end 7.8 0.19) (layer "F.Fab") (width 0.1))
-    (fp_line (start -8.05 -1.06) (end -8.6 -1.06) (layer "F.Fab") (width 0.1))
-    (fp_line (start -6 -0.71) (end -5.5 0.04) (layer "F.Fab") (width 0.1))
-    (fp_line (start -8.05 -0.71) (end -8.05 -1.06) (layer "F.Fab") (width 0.1))
-    (fp_line (start -7.8 4.19) (end 7.8 4.19) (layer "F.Fab") (width 0.1))
-    (fp_line (start 8.6 2.89) (end 8.6 -1.06) (layer "F.Fab") (width 0.1))
-    (fp_line (start -5.5 0.04) (end -5 -0.71) (layer "F.Fab") (width 0.1))
-    (fp_line (start 8.05 -1.06) (end 8.05 -0.71) (layer "F.Fab") (width 0.1))
-    (fp_line (start -7.8 0.19) (end -7.8 4.19) (layer "F.Fab") (width 0.1))
-    (fp_line (start -8.6 -1.06) (end -8.6 2.89) (layer "F.Fab") (width 0.1))
-    (fp_line (start 8.6 -1.06) (end 8.05 -1.06) (layer "F.Fab") (width 0.1))
-    (fp_line (start -8.6 2.89) (end 8.6 2.89) (layer "F.Fab") (width 0.1))
-    (pad "1" smd rect (at -5.5 -0.91) (size 0.4 1) (layers "F.Cu" "F.Paste" "F.Mask")
+    (pad "1" smd roundrect (at -5.5 -1) (size 0.6 1.3) (layers "F.Cu" "F.Paste" "F.Mask") (roundrect_rratio 0.25)
       (net 10 "GP1") (pinfunction "Pin_1") (pintype "passive"))
-    (pad "2" smd rect (at -4.5 -0.91) (size 0.4 1) (layers "F.Cu" "F.Paste" "F.Mask")
+    (pad "2" smd roundrect (at -4.5 -1) (size 0.6 1.3) (layers "F.Cu" "F.Paste" "F.Mask") (roundrect_rratio 0.25)
       (net 11 "GP2") (pinfunction "Pin_2") (pintype "passive"))
-    (pad "3" smd rect (at -3.5 -0.91) (size 0.4 1) (layers "F.Cu" "F.Paste" "F.Mask")
+    (pad "3" smd roundrect (at -3.5 -1) (size 0.6 1.3) (layers "F.Cu" "F.Paste" "F.Mask") (roundrect_rratio 0.25)
       (net 12 "GP3") (pinfunction "Pin_3") (pintype "passive"))
-    (pad "4" smd rect (at -2.5 -0.91) (size 0.4 1) (layers "F.Cu" "F.Paste" "F.Mask")
+    (pad "4" smd roundrect (at -2.5 -1) (size 0.6 1.3) (layers "F.Cu" "F.Paste" "F.Mask") (roundrect_rratio 0.25)
       (net 13 "GP4") (pinfunction "Pin_4") (pintype "passive"))
-    (pad "5" smd rect (at -1.5 -0.91) (size 0.4 1) (layers "F.Cu" "F.Paste" "F.Mask")
+    (pad "5" smd roundrect (at -1.5 -1) (size 0.6 1.3) (layers "F.Cu" "F.Paste" "F.Mask") (roundrect_rratio 0.25)
       (net 14 "GP5") (pinfunction "Pin_5") (pintype "passive"))
-    (pad "6" smd rect (at -0.5 -0.91) (size 0.4 1) (layers "F.Cu" "F.Paste" "F.Mask")
+    (pad "6" smd roundrect (at -0.5 -1) (size 0.6 1.3) (layers "F.Cu" "F.Paste" "F.Mask") (roundrect_rratio 0.25)
       (net 15 "GP6") (pinfunction "Pin_6") (pintype "passive"))
-    (pad "7" smd rect (at 0.5 -0.91) (size 0.4 1) (layers "F.Cu" "F.Paste" "F.Mask")
+    (pad "7" smd roundrect (at 0.5 -1) (size 0.6 1.3) (layers "F.Cu" "F.Paste" "F.Mask") (roundrect_rratio 0.25)
       (net 16 "GP7") (pinfunction "Pin_7") (pintype "passive"))
-    (pad "8" smd rect (at 1.5 -0.91) (size 0.4 1) (layers "F.Cu" "F.Paste" "F.Mask")
+    (pad "8" smd roundrect (at 1.5 -1) (size 0.6 1.3) (layers "F.Cu" "F.Paste" "F.Mask") (roundrect_rratio 0.25)
       (net 17 "GP8") (pinfunction "Pin_8") (pintype "passive"))
-    (pad "9" smd rect (at 2.5 -0.91) (size 0.4 1) (layers "F.Cu" "F.Paste" "F.Mask")
+    (pad "9" smd roundrect (at 2.5 -1) (size 0.6 1.3) (layers "F.Cu" "F.Paste" "F.Mask") (roundrect_rratio 0.25)
       (net 18 "GP9") (pinfunction "Pin_9") (pintype "passive"))
-    (pad "10" smd rect (at 3.5 -0.91) (size 0.4 1) (layers "F.Cu" "F.Paste" "F.Mask")
+    (pad "10" smd roundrect (at 3.5 -1) (size 0.6 1.3) (layers "F.Cu" "F.Paste" "F.Mask") (roundrect_rratio 0.25)
       (net 21 "GP10") (pinfunction "Pin_10") (pintype "passive"))
-    (pad "11" smd rect (at 4.5 -0.91) (size 0.4 1) (layers "F.Cu" "F.Paste" "F.Mask")
+    (pad "11" smd roundrect (at 4.5 -1) (size 0.6 1.3) (layers "F.Cu" "F.Paste" "F.Mask") (roundrect_rratio 0.25)
       (net 20 "GP11") (pinfunction "Pin_11") (pintype "passive"))
-    (pad "12" smd rect (at 5.5 -0.91) (size 0.4 1) (layers "F.Cu" "F.Paste" "F.Mask")
+    (pad "12" smd roundrect (at 5.5 -1) (size 0.6 1.3) (layers "F.Cu" "F.Paste" "F.Mask") (roundrect_rratio 0.25)
       (net 19 "GP12") (pinfunction "Pin_12") (pintype "passive"))
-    (pad "MP" smd rect (at -8.3 1.79) (size 2 1.3) (layers "F.Cu" "F.Paste" "F.Mask"))
-    (pad "MP" smd rect (at 8.3 1.79) (size 2 1.3) (layers "F.Cu" "F.Paste" "F.Mask"))
-    (model "${KICAD6_3DMODEL_DIR}/Connector_FFC-FPC.3dshapes/Molex_200528-0120_1x12-1MP_P1.00mm_Horizontal.wrl"
-      (offset (xyz 0 0 0))
-      (scale (xyz 1 1 1))
-      (rotate (xyz 0 0 0))
-    )
+    (pad "MP" smd roundrect (at -8.1 2.25) (size 1 2) (layers "F.Cu" "F.Paste" "F.Mask") (roundrect_rratio 0.25))
+    (pad "MP" smd roundrect (at 8.1 2.25) (size 1 2) (layers "F.Cu" "F.Paste" "F.Mask") (roundrect_rratio 0.25))
   )
   (footprint "Connector_JST:JST_SH_SM04B-SRSS-TB_1x04-1MP_P1.00mm_Horizontal" (layer "F.Cu")
