File: PCB/rp2040_zero_controller/rp2040_zero.kicad_sch (KiCad schematic)
At the start: 15 parts, among them J1 Conn_01x04, J2 Conn_01x04, J3 Conn_01x04, J4 Conn_01x12, J5 Conn_01x04, U1 rp2040_zero, U2 74AHCT1G125, U3 74AHCT1G125

Commit message: temp
Parts:
- removed H? (x2): MountingHole, MountingHole:MountingHole_2.1mm, symbol Mechanical:MountingHole
- removed U3: 74AHCT1G125, Package_TO_SOT_SMD:SOT-23-5_HandSoldering, symbol 74xGxx:74AHCT1G126
- J4: footprint ergodash_controller:HDGC_1.0K-J-12PW -> Connector_FFC-FPC:Molex_200528-0120_1x12-1MP_P1.00mm_Horizontal
Connections:
- net RGB_5v is gone; now on net SCL: J2.4 (Pin_4)
- net +3V3: now also R3.1; no longer R3.2
- net GP1: now also U1.26; no longer U1.13
- net GP10: now also U1.7; no longer U1.9
- net GP11: now also U1.6; no longer U1.7
- net GP12: now also U1.5; no longer U1.8
- net GP2: now also U1.15; no longer U1.14
- net GP3: now also U1.14; no longer U1.12
- net GP4: now also U1.13; no longer U1.15
- net GP5: now also U1.12; no longer U1.11
- net GP6: now also U1.11; no longer U1.26
- net GP7: now also U1.10; no longer U1.5
- net GP8: now also U1.9; no longer U1.10
- net GP9: now also U1.8; no longer U1.6
- net Handness: now also R3.2, U1.27; no longer R3.1, U1.28
- net RGB: now also U2.2
- net RGB_5v_2: now also J1.4 (Pin_4)
- net SCL: now also R1.2; no longer J1.4 (Pin_4), R2.2
- net SDA: now also J2.3 (Pin_3), R2.2; no longer J1.3 (Pin_3), R1.2
- net VCC: now also J1.3 (Pin_3); no longer J2.3 (Pin_3)
- removed net RGB2: U1.27, U2.2

Commit message: temp
Parts:
- J4: footprint Connector_FFC-FPC:Molex_200528-0120_1x12-1MP_P1.00mm_Horizontal -> ergodash_controller:CF50121D0R0-10-NH
Changed lines of the file:
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@@
     (property "Reference" "J4" (id 0) (at 193.04 53.34 0))
     (property "Value" "Conn_01x12" (id 1) (at 193.04 55.88 0))
-    (property "Footprint" "Connector_FFC-FPC:Molex_200528-0120_1x12-1MP_P1.00mm_Horizontal" (id 2) (at 193.04 72.39 0)
+    (property "Footprint" "ergodash_controller:CF50121D0R0-10-NH" (id 2) (at 193.04 72.39 0)
       (effects (font (size 1.27 1.27)) hide)
     )
@@
     )
     (path "/0d38d324-03a5-4b0b-9014-dff533b56cd1"
-      (reference "J4") (unit 1) (value "Conn_01x12") (footprint "Connector_FFC-FPC:Molex_200528-0120_1x12-1MP_P1.00mm_Horizontal")
+      (reference "J4") (unit 1) (value "Conn_01x12") (footprint "ergodash_controller:CF50121D0R0-10-NH")
     )
     (path "/13c35b16-c113-41c3-811d-ca2cd7617f5a"

Commit message: firmware temp
Other:
- note removed: "GPIO07"
- note removed: "GPIO08"
- note removed: "GPIO09"
- note removed: "GPIO16"
- note removed: "GPIO17"
- note removed: "GPIO18"
- note removed: "GPIO19"
- note removed: "GPIO20"
- note removed: "GPIO21"
- note removed: "GPIO22"
- note removed: "GPIO26"
- note removed: "GPIO27"
Changed lines of the file:
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@@
     (stroke (width 0) (type default) (color 0 0 0 0))
-  )
-  (text "GPIO27" (at 204.47 60.96 0)
-    (effects (font (size 1.27 1.27)) (justify left bottom))
-  )
-  (text "GPIO08" (at 205.74 86.36 0)
-    (effects (font (size 1.27 1.27)) (justify left bottom))
-  )
-  (text "GPIO22" (at 204.47 66.04 0)
-    (effects (font (size 1.27 1.27)) (justify left bottom))
-  )
-  (text "GPIO18" (at 204.47 76.2 0)
-    (effects (font (size 1.27 1.27)) (justify left bottom))
-  )
-  (text "GPIO21" (at 204.47 68.58 0)
-    (effects (font (size 1.27 1.27)) (justify left bottom))
-  )
-  (text "GPIO20" (at 204.47 71.12 0)
-    (effects (font (size 1.27 1.27)) (justify left bottom))
-  )
-  (text "GPIO17" (at 204.47 78.74 0)
-    (effects (font (size 1.27 1.27)) (justify left bottom))
-  )
-  (text "GPIO16" (at 204.47 81.28 0)
-    (effects (font (size 1.27 1.27)) (justify left bottom))
-  )
-  (text "GPIO26\n" (at 204.47 63.5 0)
-    (effects (font (size 1.27 1.27)) (justify left bottom))
-  )
-  (text "GPIO19" (at 204.47 73.66 0)
-    (effects (font (size 1.27 1.27)) (justify left bottom))
-  )
-  (text "GPIO07" (at 205.74 83.82 0)
-    (effects (font (size 1.27 1.27)) (justify left bottom))
-  )
-  (text "GPIO09" (at 205.74 88.9 0)
-    (effects (font (size 1.27 1.27)) (justify left bottom))
   )
   (global_label "RGB_5v_2" (shape input) (at 102.87 190.5 0) (fields_autoplaced)
